Commit message: Simplify D435 in GO1 URDF to a single visualization-only link
The full realsense-ros frame tree (bottom_screw_frame + 8 optical frames) is
unused for IsaacLab: those empty frames merge away under merge_fixed_joints=True,
and the DAGGER depth sensor mounts on the base body with an offset. Keep only
d435_link (mesh visual) mounted on trunk for visualization; drop its
collision/inertial so it adds no mass and no physics.

Co-Authored-By: Claude <noreply@anthropic.com>

File: source/basic_locomotion_isaaclab/basic_locomotion_isaaclab/assets/go1_asset/urdf/go1.urdf (robot description, URDF)
Before this commit: robot go1_description, 48 links, 47 joints
Links:
- removed link d435_bottom_screw_frame
- removed link d435_color_frame
- removed link d435_color_optical_frame
- removed link d435_depth_frame
- removed link d435_depth_optical_frame
- removed link d435_infra1_frame
- removed link d435_infra1_optical_frame
- removed link d435_infra2_frame
- removed link d435_infra2_optical_frame
- link d435_link: mass 0.072 -> None; geometry visual mesh filename=../meshes/d435.dae scale=1 1 1
Joints:
- removed joint d435_color_joint
- removed joint d435_color_optical_joint
- removed joint d435_depth_joint
- removed joint d435_depth_optical_joint
- removed joint d435_infra1_joint
- removed joint d435_infra1_optical_joint
- removed joint d435_infra2_joint
- removed joint d435_infra2_optical_joint
- removed joint d435_link_joint
- joint d435_joint: child d435_bottom_screw_frame -> d435_link

Commit message: Restore D435 mount frame (bottom_screw_frame) as mechanical reference
Keep the d435_bottom_screw_frame + d435_link_joint structure so the mount pose
(trunk -> screw mount) is an explicit frame in the URDF; the 3D-printed bracket
only needs to realize that single trunk<->screw-mount relative pose. The camera
body (d435_link) stays visualization-only with no collision/inertial.

Co-Authored-By: Claude <noreply@anthropic.com>

File: source/basic_locomotion_isaaclab/basic_locomotion_isaaclab/assets/go1_asset/urdf/go1.urdf (robot description, URDF)
Before this commit: robot go1_description, 39 links, 38 joints
Links:
- added link d435_bottom_screw_frame
Joints:
- added joint d435_link_joint: type fixed, parent d435_bottom_screw_frame, child d435_link, origin xyz=0.0106 0.0175 0.0125 rpy=0 0 0
- joint d435_joint: child d435_link -> d435_bottom_screw_frame

Commit message: GO1 Tiled env: fix D435 camera pose and terrain curriculum
- URDF d435_joint moved to (0.26, 0, 0.12) to reduce the head appearing in the
  depth image; TiledCamera offset pos matches.
- TiledCamera offset rot changed from the reference 20-deg quaternion to the
  true 30-deg-down + upright one ((-0.353553, 0.612372, -0.612372, 0.353553)),
  computed and validated by reproducing the reference quaternion at 20 deg.
- Tiled terrain curriculum forced False: with enforce_env_spacing (one robot
  fixed per sub-terrain) the curriculum's update_env_origins would move envs to
  random sub-terrains -> overlaps -> physics crashes (matches reference M1/Aliengo).

Co-Authored-By: Claude <noreply@anthropic.com>

File: source/basic_locomotion_isaaclab/basic_locomotion_isaaclab/assets/go1_asset/urdf/go1.urdf (robot description, URDF)
Before this commit: robot go1_description, 40 links, 39 joints
Joints:
- joint d435_joint: origin xyz=0.23 0.0 0.10 rpy=0 0.5235987755982988 0 -> xyz=0.26 0.0 0.12 rpy=0 0.5235987755982988 0

Commit message: GO1 dagger: comment out D435 camera-body visual, add student-depth dual-pane option
The D435 camera body mesh in go1.urdf sat exactly at the depth camera's mount,
so the rendered depth saw the camera's own housing as a big near-field white
blob. Commented the visual out (kept for later visualization); camera stays at
the URDF d435 pose (0.26, 0, 0.12, 30 deg down, 87 deg HFOV).

train_dagger_go1.py: new --dual_pane_student_depth shows the right pane as the
student's actual sanitized depth input (clip [0.1, 2.0], no-hit -> 1.0) instead
of the raw camera depth, for verifying what the student obs really receives.

Co-Authored-By: Claude <noreply@anthropic.com>

File: source/basic_locomotion_isaaclab/basic_locomotion_isaaclab/assets/go1_asset/urdf/go1.urdf (robot description, URDF)
Before this commit: robot go1_description, 40 links, 39 joints
Links:
- link d435_link: geometry 
