Commit message: tune: finetune d435 position

File: source/basic_locomotion_isaaclab/basic_locomotion_isaaclab/assets/go1_asset/urdf/go1.urdf (robot description, URDF)
Before this commit: robot go1_description, 40 links, 39 joints
Joints:
- joint d435_joint: origin xyz=0.28 0.0 0.08 rpy=0 0.5235987755982988 0 -> xyz=0.23 0.0 0.10 rpy=0 0.5235987755982988 0

Commit message: fix(go1): align asset with Unitree URDF
Replace the local Go1 model with Unitree's official URDF so joint position, velocity and effort limits, link masses, inertias and collisions match the upstream robot description.

Keep only the IsaacLab-specific adaptations: resolve meshes from the bundled asset directory and preserve the four foot bodies with dont_collapse for contact sensing. Regenerate the feet-only collision variant from the same source.

Remove duplicated actuator effort and velocity overrides so the URDF is the single source of truth, and extend the asset smoke test to validate official limits, body names and the 13.1005 kg merged mass.

File: source/basic_locomotion_isaaclab/basic_locomotion_isaaclab/assets/go1_asset/urdf/go1.urdf (robot description, URDF)
Before this commit: robot go1_description, 40 links, 39 joints
Links:
- removed link FL_thigh_shoulder
- removed link FR_thigh_shoulder
- removed link RL_thigh_shoulder
- removed link RR_thigh_shoulder
- removed link d435_bottom_screw_frame
- removed link d435_link
- added link FL_calf_rotor, mass 0.089; collision cylinder length=0.02 radius=0.035; visual cylinder length=0.02 radius=0.035
- added link FL_hip_rotor, mass 0.089; collision cylinder length=0.02 radius=0.035; visual cylinder length=0.02 radius=0.035
- added link FL_thigh_rotor, mass 0.089; collision cylinder length=0.02 radius=0.035; visual cylinder length=0.02 radius=0.035
- added link FR_calf_rotor, mass 0.089; collision cylinder length=0.02 radius=0.035; visual cylinder length=0.02 radius=0.035
- added link FR_hip_rotor, mass 0.089; collision cylinder length=0.02 radius=0.035; visual cylinder length=0.02 radius=0.035
- added link FR_thigh_rotor, mass 0.089; collision cylinder length=0.02 radius=0.035; visual cylinder length=0.02 radius=0.035
- added link RL_calf_rotor, mass 0.089; collision cylinder length=0.02 radius=0.035; visual cylinder length=0.02 radius=0.035
- added link RL_hip_rotor, mass 0.089; collision cylinder length=0.02 radius=0.035; visual cylinder length=0.02 radius=0.035
- added link RL_thigh_rotor, mass 0.089; collision cylinder length=0.02 radius=0.035; visual cylinder length=0.02 radius=0.035
- added link RR_calf_rotor, mass 0.089; collision cylinder length=0.02 radius=0.035; visual cylinder length=0.02 radius=0.035
- added link RR_hip_rotor, mass 0.089; collision cylinder length=0.02 radius=0.035; visual cylinder length=0.02 radius=0.035
- added link RR_thigh_rotor, mass 0.089; collision cylinder length=0.02 radius=0.035; visual cylinder length=0.02 radius=0.035
- link FL_calf: mass 0.158015 -> 0.135862
- link FL_hip: mass 0.510299 -> 0.591; geometry collision cylinder length=0.04 radius=0.046; visual mesh filename=../meshes/hip.dae scale=1 1 1
- link FL_thigh: mass 0.898919 -> 0.92
- link FR_calf: mass 0.158015 -> 0.135862
- link FR_hip: mass 0.510299 -> 0.591; geometry collision cylinder length=0.04 radius=0.046; visual mesh filename=../meshes/hip.dae scale=1 1 1
- link FR_thigh: mass 0.898919 -> 0.92
- link RL_calf: mass 0.158015 -> 0.135862
- link RL_hip: mass 0.510299 -> 0.591; geometry collision cylinder length=0.04 radius=0.046; visual mesh filename=../meshes/hip.dae scale=1 1 1
- link RL_thigh: mass 0.898919 -> 0.92
- link RR_calf: mass 0.158015 -> 0.135862
- link RR_hip: mass 0.510299 -> 0.591; geometry collision cylinder length=0.04 radius=0.046; visual mesh filename=../meshes/hip.dae scale=1 1 1
- link RR_thigh: mass 0.898919 -> 0.92
- link trunk: mass 4.8 -> 5.204; geometry collision box size=0.3762 0.0935 0.114; visual mesh filename=../meshes/trunk.dae scale=1 1 1
Joints:
- removed joint FL_hip_fixed
- removed joint FR_hip_fixed
- removed joint RL_hip_fixed
- removed joint RR_hip_fixed
- removed joint d435_joint
- removed joint d435_link_joint
- added joint FL_calf_rotor_joint: type fixed, parent FL_thigh, child FL_calf_rotor, origin xyz=0.0 -0.03235 0 rpy=0 0 0
- added joint FL_hip_rotor_joint: type fixed, parent trunk, child FL_hip_rotor, origin xyz=0.11215 0.04675 0 rpy=0 0 0
- added joint FL_thigh_rotor_joint: type fixed, parent FL_hip, child FL_thigh_rotor, origin xyz=0.0 -0.00015 0 rpy=0 0 0
- added joint FR_calf_rotor_joint: type fixed, parent FR_thigh, child FR_calf_rotor, origin xyz=0.0 0.03235 0 rpy=0 0 0
- added joint FR_hip_rotor_joint: type fixed, parent trunk, child FR_hip_rotor, origin xyz=0.11215 -0.04675 0 rpy=0 0 0
- added joint FR_thigh_rotor_joint: type fixed, parent FR_hip, child FR_thigh_rotor, origin xyz=0.0 0.00015 0 rpy=0 0 0
- added joint RL_calf_rotor_joint: type fixed, parent RL_thigh, child RL_calf_rotor, origin xyz=0.0 -0.03235 0 rpy=0 0 0
- added joint RL_hip_rotor_joint: type fixed, parent trunk, child RL_hip_rotor, origin xyz=-0.11215 0.04675 0 rpy=0 0 0
- added joint RL_thigh_rotor_joint: type fixed, parent RL_hip, child RL_thigh_rotor, origin xyz=0.0 -0.00015 0 rpy=0 0 0
- added joint RR_calf_rotor_joint: type fixed, parent RR_thigh, child RR_calf_rotor, origin xyz=0.0 0.03235 0 rpy=0 0 0
- added joint RR_hip_rotor_joint: type fixed, parent trunk, child RR_hip_rotor, origin xyz=-0.11215 -0.04675 0 rpy=0 0 0
- added joint RR_thigh_rotor_joint: type fixed, parent RR_hip, child RR_thigh_rotor, origin xyz=0.0 0.00015 0 rpy=0 0 0
- joint FL_calf_joint: limit lower=-2.6965336943312392 upper=-0.9162978572970231 effort=33.5 velocity=21 -> lower=-2.818 upper=-0.888 effort=35.55 velocity=20.06
- joint FL_hip_joint: limit lower=-0.8028514559173915 upper=0.8028514559173915 effort=33.5 velocity=21 -> lower=-0.863 upper=0.863 effort=23.7 velocity=30.1
- joint FL_thigh_joint: limit lower=-1.0471975511965976 upper=4.1887902047863905 effort=33.5 velocity=21 -> lower=-0.686 upper=4.501 effort=23.7 velocity=30.1
- joint FR_calf_joint: limit lower=-2.6965336943312392 upper=-0.9162978572970231 effort=33.5 velocity=21 -> lower=-2.818 upper=-0.888 effort=35.55 velocity=20.06
- joint FR_hip_joint: limit lower=-0.8028514559173915 upper=0.8028514559173915 effort=33.5 velocity=21 -> lower=-0.863 upper=0.863 effort=23.7 velocity=30.1
- joint FR_thigh_joint: limit lower=-1.0471975511965976 upper=4.1887902047863905 effort=33.5 velocity=21 -> lower=-0.686 upper=4.501 effort=23.7 velocity=30.1
- joint RL_calf_joint: limit lower=-2.6965336943312392 upper=-0.9162978572970231 effort=33.5 velocity=21 -> lower=-2.818 upper=-0.888 effort=35.55 velocity=20.06
- joint RL_hip_joint: limit lower=-0.8028514559173915 upper=0.8028514559173915 effort=33.5 velocity=21 -> lower=-0.863 upper=0.863 effort=23.7 velocity=30.1
- joint RL_thigh_joint: limit lower=-1.0471975511965976 upper=4.1887902047863905 effort=33.5 velocity=21 -> lower=-0.686 upper=4.501 effort=23.7 velocity=30.1
- joint RR_calf_joint: limit lower=-2.6965336943312392 upper=-0.9162978572970231 effort=33.5 velocity=21 -> lower=-2.818 upper=-0.888 effort=35.55 velocity=20.06
- joint RR_hip_joint: limit lower=-0.8028514559173915 upper=0.8028514559173915 effort=33.5 velocity=21 -> lower=-0.863 upper=0.863 effort=23.7 velocity=30.1
- joint RR_thigh_joint: limit lower=-1.0471975511965976 upper=4.1887902047863905 effort=33.5 velocity=21 -> lower=-0.686 upper=4.501 effort=23.7 velocity=30.1

File: source/basic_locomotion_isaaclab/basic_locomotion_isaaclab/assets/go1_asset/urdf/go1_feetonly.urdf (robot description, URDF)
Before this commit: robot go1_description, 40 links, 39 joints
Links:
- removed link FL_thigh_shoulder
- removed link FR_thigh_shoulder
- removed link RL_thigh_shoulder
- removed link RR_thigh_shoulder
- removed link d435_bottom_screw_frame
- removed link d435_link
- added link FL_calf_rotor, mass 0.089; visual cylinder length=0.02 radius=0.035
- added link FL_hip_rotor, mass 0.089; visual cylinder length=0.02 radius=0.035
- added link FL_thigh_rotor, mass 0.089; visual cylinder length=0.02 radius=0.035
- added link FR_calf_rotor, mass 0.089; visual cylinder length=0.02 radius=0.035
- added link FR_hip_rotor, mass 0.089; visual cylinder length=0.02 radius=0.035
- added link FR_thigh_rotor, mass 0.089; visual cylinder length=0.02 radius=0.035
- added link RL_calf_rotor, mass 0.089; visual cylinder length=0.02 radius=0.035
- added link RL_hip_rotor, mass 0.089; visual cylinder length=0.02 radius=0.035
- added link RL_thigh_rotor, mass 0.089; visual cylinder length=0.02 radius=0.035
- added link RR_calf_rotor, mass 0.089; visual cylinder length=0.02 radius=0.035
- added link RR_hip_rotor, mass 0.089; visual cylinder length=0.02 radius=0.035
- added link RR_thigh_rotor, mass 0.089; visual cylinder length=0.02 radius=0.035
- link FL_calf: mass 0.158015 -> 0.135862
- link FL_hip: mass 0.510299 -> 0.591
- link FL_thigh: mass 0.898919 -> 0.92
- link FR_calf: mass 0.158015 -> 0.135862
- link FR_hip: mass 0.510299 -> 0.591
- link FR_thigh: mass 0.898919 -> 0.92
- link RL_calf: mass 0.158015 -> 0.135862
- link RL_hip: mass 0.510299 -> 0.591
- link RL_thigh: mass 0.898919 -> 0.92
- link RR_calf: mass 0.158015 -> 0.135862
- link RR_hip: mass 0.510299 -> 0.591
- link RR_thigh: mass 0.898919 -> 0.92
- link trunk: mass 4.8 -> 5.204
Joints:
- removed joint FL_hip_fixed
- removed joint FR_hip_fixed
- removed joint RL_hip_fixed
- removed joint RR_hip_fixed
- removed joint d435_joint
- removed joint d435_link_joint
- added joint FL_calf_rotor_joint: type fixed, parent FL_thigh, child FL_calf_rotor, origin xyz=0.0 -0.03235 0 rpy=0 0 0
- added joint FL_hip_rotor_joint: type fixed, parent trunk, child FL_hip_rotor, origin xyz=0.11215 0.04675 0 rpy=0 0 0
- added joint FL_thigh_rotor_joint: type fixed, parent FL_hip, child FL_thigh_rotor, origin xyz=0.0 -0.00015 0 rpy=0 0 0
- added joint FR_calf_rotor_joint: type fixed, parent FR_thigh, child FR_calf_rotor, origin xyz=0.0 0.03235 0 rpy=0 0 0
- added joint FR_hip_rotor_joint: type fixed, parent trunk, child FR_hip_rotor, origin xyz=0.11215 -0.04675 0 rpy=0 0 0
- added joint FR_thigh_rotor_joint: type fixed, parent FR_hip, child FR_thigh_rotor, origin xyz=0.0 0.00015 0 rpy=0 0 0
- added joint RL_calf_rotor_joint: type fixed, parent RL_thigh, child RL_calf_rotor, origin xyz=0.0 -0.03235 0 rpy=0 0 0
- added joint RL_hip_rotor_joint: type fixed, parent trunk, child RL_hip_rotor, origin xyz=-0.11215 0.04675 0 rpy=0 0 0
- added joint RL_thigh_rotor_joint: type fixed, parent RL_hip, child RL_thigh_rotor, origin xyz=0.0 -0.00015 0 rpy=0 0 0
- added joint RR_calf_rotor_joint: type fixed, parent RR_thigh, child RR_calf_rotor, origin xyz=0.0 0.03235 0 rpy=0 0 0
- added joint RR_hip_rotor_joint: type fixed, parent trunk, child RR_hip_rotor, origin xyz=-0.11215 -0.04675 0 rpy=0 0 0
- added joint RR_thigh_rotor_joint: type fixed, parent RR_hip, child RR_thigh_rotor, origin xyz=0.0 0.00015 0 rpy=0 0 0
- joint FL_calf_joint: limit lower=-2.6965336943312392 upper=-0.9162978572970231 effort=33.5 velocity=21 -> lower=-2.818 upper=-0.888 effort=35.55 velocity=20.06
- joint FL_hip_joint: limit lower=-0.8028514559173915 upper=0.8028514559173915 effort=33.5 velocity=21 -> lower=-0.863 upper=0.863 effort=23.7 velocity=30.1
- joint FL_thigh_joint: limit lower=-1.0471975511965976 upper=4.1887902047863905 effort=33.5 velocity=21 -> lower=-0.686 upper=4.501 effort=23.7 velocity=30.1
- joint FR_calf_joint: limit lower=-2.6965336943312392 upper=-0.9162978572970231 effort=33.5 velocity=21 -> lower=-2.818 upper=-0.888 effort=35.55 velocity=20.06
- joint FR_hip_joint: limit lower=-0.8028514559173915 upper=0.8028514559173915 effort=33.5 velocity=21 -> lower=-0.863 upper=0.863 effort=23.7 velocity=30.1
- joint FR_thigh_joint: limit lower=-1.0471975511965976 upper=4.1887902047863905 effort=33.5 velocity=21 -> lower=-0.686 upper=4.501 effort=23.7 velocity=30.1
- joint RL_calf_joint: limit lower=-2.6965336943312392 upper=-0.9162978572970231 effort=33.5 velocity=21 -> lower=-2.818 upper=-0.888 effort=35.55 velocity=20.06
- joint RL_hip_joint: limit lower=-0.8028514559173915 upper=0.8028514559173915 effort=33.5 velocity=21 -> lower=-0.863 upper=0.863 effort=23.7 velocity=30.1
- joint RL_thigh_joint: limit lower=-1.0471975511965976 upper=4.1887902047863905 effort=33.5 velocity=21 -> lower=-0.686 upper=4.501 effort=23.7 velocity=30.1
- joint RR_calf_joint: limit lower=-2.6965336943312392 upper=-0.9162978572970231 effort=33.5 velocity=21 -> lower=-2.818 upper=-0.888 effort=35.55 velocity=20.06
- joint RR_hip_joint: limit lower=-0.8028514559173915 upper=0.8028514559173915 effort=33.5 velocity=21 -> lower=-0.863 upper=0.863 effort=23.7 velocity=30.1
- joint RR_thigh_joint: limit lower=-1.0471975511965976 upper=4.1887902047863905 effort=33.5 velocity=21 -> lower=-0.686 upper=4.501 effort=23.7 velocity=30.1
